File: RoboKit/RoboKit.sch (EAGLE design)
At the start: 27 parts, among them CON1 XT30UPB-M, CON2 XT30UPB-M, P1 B6B-PH-K, P2 B6B-PH-K, U1 SSM6J808R, X1 JST-XH-06-PIN-LONG-PAD, X2 JST-XH-06-PIN-LONG-PAD, X3 JST-XH-02-PIN-LONG-PAD, X4 JST-XH-02-PIN-LONG-PAD, X5 JST-XH-04-PIN-LONG-PAD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

Commit message: make_circuit
Parts:
- removed X1, X2: JST-XH-06-PIN-LONG-PAD, JST XH Connectors:JST-XH-06-PIN-LONG-PAD
- added CONNECTOR1: RESISTER, resistor:RESISTER
- added S1: (no value), switch-omron:10-XX
- added TC4052DP: (no value), ic-package:DIL16
- added X7: JST-XH-10-PIN-LONG-PAD, Rembrandt Electronics - JST XH Connectors v1-0:JST-XH-10-PIN-LONG-PAD
- added X8: JST-XH-02-PIN-LONG-PAD, Rembrandt Electronics - JST XH Connectors v1-0:JST-XH-02-PIN-LONG-PAD
- added X9: JST-XH-03-PIN-LONG-PAD, Rembrandt Electronics - JST XH Connectors v1-0:JST-XH-03-PIN-LONG-PAD
Connections:
- removed net +5V: X1-2.S, X2-2.S
- removed net ADC0: U$1.31
- removed net ADC1: U$1.32
- removed net IO16: U$1.21
- removed net IO17: U$1.22
- removed net LINE: X1-3.S, X2-3.S
- removed net MD_INA_L: U$2.AIN1, U$2.AIN2
- removed net MD_INA_R: U$3.AIN1, U$3.AIN2
- removed net MD_INB_L: U$2.BIN1, U$2.BIN2
- removed net MD_INB_R: U$3.BIN1, U$3.BIN2
- removed net MOTER_A_L: X3-1.S
- removed net MOTER_A_R: X4-1.S
- removed net MOTER_B_L: X3-2.S
- removed net MOTER_B_R: X4-2.S
- removed net MUX0: X1-4.S, X2-4.S
- removed net MUX1: X1-5.S, X2-5.S
- removed net MUX2: X1-6.S, X2-6.S
- new net 0X: TC4052DP.12, X7-3.S
- new net 0Y: TC4052DP.1, X7-7.S
- new net 1X: TC4052DP.14, X7-4.S
- new net 1Y: TC4052DP.5, X7-8.S
- new net 2X: TC4052DP.15, X7-5.S
- new net 2Y: TC4052DP.2, X7-9.S
- new net 3X: TC4052DP.11, X7-6.S
- new net 3Y: TC4052DP.4, X7-10.S
- new net A: TC4052DP.10, U$1.21
- new net B: TC4052DP.9, U$1.22
- new net N$4: CONNECTOR1.2, S1.P
- new net X-COM: TC4052DP.13, U$1.32
- new net Y-COM: TC4052DP.3, U$1.31
- net 3V3: now also CONNECTOR1.1
- net GND: now also S1.S1, TC4052DP.6, TC4052DP.7, TC4052DP.8, X7-1.S, X8-2.S, X9-2.S; no longer X1-1.S, X2-1.S
- net IO0: now also U$2.AIN1, U$2.BIN1
- net IO1: now also U$2.AIN2, U$2.BIN2
- net IO2: now also U$3.AIN1, U$3.BIN1
- net IO21: now also S1.P1
- net IO3: now also U$3.AIN2, U$3.BIN2
- net IO7: now also X8-1.S
- net MOTOR_A_L: now also X3-1.S
- net MOTOR_A_R: now also X4-1.S
- net MOTOR_B_L: now also X3-2.S
- net MOTOR_B_R: now also X4-2.S
- net VBUS: now also TC4052DP.16, X7-2.S, X9-1.S
- net VOUT: now also X9-3.S

Commit message: make_okunishi_1
Connections:
- net 3V3_EN: now also X6-1.S
- net VCC: no longer X6-1.S
Changed lines of the file:
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@@
 <label x="40.64" y="60.96" size="0.762" layer="95" xref="yes"/>
+</segment>
+<segment>
+<pinref part="X6" gate="-1" pin="S"/>
+<wire x1="101.6" y1="83.82" x2="99.06" y2="83.82" width="0.1524" layer="91"/>
+<label x="99.06" y="83.82" size="1.778" layer="95" rot="R180" xref="yes"/>
 </segment>
 </net>
@@
 <label x="20.32" y="91.44" size="0.762" layer="95" rot="R180" xref="yes"/>
 </segment>
-<segment>
-<pinref part="X6" gate="-1" pin="S"/>
-<wire x1="101.6" y1="83.82" x2="99.06" y2="83.82" width="0.1524" layer="91"/>
-<label x="99.06" y="83.82" size="1.778" layer="95" rot="R180" xref="yes"/>
-</segment>
 </net>

Commit message: 回路図の完成
Parts:
- added S2: (no value), switch:320-916
Connections:
- removed net IO10: U$1.14
- removed net IO11: U$1.15
- removed net IO12: U$1.16
- removed net IO13: U$1.17
- removed net IO4: U$1.6
- removed net IO5: U$1.7
- new net 5.0V: S2.P, X9-1.S
- net HALL_A_L: now also U$1.16
- net HALL_A_R: now also U$1.14
- net HALL_B_L: now also U$1.17
- net HALL_B_R: now also U$1.15
- net SCL: now also U$1.7
- net SDA: now also U$1.6
- net VBUS: now also S2.S; no longer X9-1.S
Changed lines of the file:
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@@
 <part name="GND8" library="supply1" library_urn="urn:adsk.eagle:library:371" deviceset="GND" device=""/>
 <part name="X9" library="Rembrandt Electronics - JST XH Connectors v1-0" deviceset="JST-XH-03-PIN" device="-LONG-PAD"/>
+<part name="S2" library="switch" deviceset="320-916" device=""/>
 </parts>
 <sheets>
@@
 <attribute name="NAME" x="261.62" y="60.198" size="1.524" layer="95"/>
 </instance>
+<instance part="S2" gate="1" x="266.7" y="81.28" smashed="yes">
+<attribute name="NAME" x="260.35" y="79.375" size="1.778" layer="95" rot="R90"/>
+<attribute name="VALUE" x="262.89" y="83.82" size="1.778" layer="96" rot="R90"/>
+</instance>
 </instances>
 <busses>
@@
 </segment>
 </net>
-<net name="IO4" class="0">
-<segment>
-<wire x1="7.62" y1="55.88" x2="5.08" y2="55.88" width="0.1524" layer="91"/>
-<pinref part="U$1" gate="G$1" pin="6"/>
-<label x="5.08" y="55.88" size="0.762" layer="95" rot="R180" xref="yes"/>
-</segment>
-</net>
-<net name="IO5" class="0">
-<segment>
-<wire x1="7.62" y1="53.34" x2="5.08" y2="53.34" width="0.1524" layer="91"/>
-<pinref part="U$1" gate="G$1" pin="7"/>
-<label x="5.08" y="53.34" size="0.762" layer="95" rot="R180" xref="yes"/>
-</segment>
-</net>
 <net name="IO6" class="0">
 <segment>
@@
 </segment>
 </net>
-<net name="IO10" class="0">
-<segment>
-<wire x1="7.62" y1="35.56" x2="5.08" y2="35.56" width="0.1524" layer="91"/>
-<pinref part="U$1" gate="G$1" pin="14"/>
-<label x="5.08" y="35.56" size="0.762" layer="95" rot="R180" xref="yes"/>
-</segment>
-</net>
-<net name="IO11" class="0">
-<segment>
-<wire x1="7.62" y1="33.02" x2="5.08" y2="33.02" width="0.1524" layer="91"/>
-<pinref part="U$1" gate="G$1" pin="15"/>
-<label x="5.08" y="33.02" size="0.762" layer="95" rot="R180" xref="yes"/>
-</segment>
-</net>
-<net name="IO12" class="0">
-<segment>
-<wire x1="7.62" y1="30.48" x2="5.08" y2="30.48" width="0.1524" layer="91"/>
-<pinref part="U$1" gate="G$1" pin="16"/>
-<label x="5.08" y="30.48" size="0.762" layer="95" rot="R180" xref="yes"/>
-</segment>
-</net>
-<net name="IO13" class="0">
-<segment>
-<wire x1="7.62" y1="27.94" x2="5.08" y2="27.94" width="0.1524" layer="91"/>
-<pinref part="U$1" gate="G$1" pin="17"/>
-<label x="5.08" y="27.94" size="0.762" layer="95" rot="R180" xref="yes"/>
-</segment>
-</net>
 <net name="IO14" class="0">
 <segment>
@@
 </segment>
 <segment>
-<pinref part="X9" gate="-1" pin="S"/>
-<wire x1="256.54" y1="66.04" x2="254" y2="66.04" width="0.1524" layer="91"/>
-<wire x1="254" y1="66.04" x2="254" y2="78.74" width="0.1524" layer="91"/>
-<label x="254" y="78.74" size="1.778" layer="95" rot="R90" xref="yes"/>
+<pinref part="S2" gate="1" pin="S"/>
+<wire x1="271.78" y1="86.36" x2="274.32" y2="86.36" width="0.1524" layer="91"/>
+<label x="274.32" y="86.36" size="1.778" layer="95" xref="yes"/>
 </segment>
 </net>
@@
 <label x="99.06" y="76.2" size="1.778" layer="95" rot="R180" xref="yes"/>
 </segment>
+<segment>
+<wire x1="7.62" y1="53.34" x2="5.08" y2="53.34" width="0.1524" layer="91"/>
+<pinref part="U$1" gate="G$1" pin="7"/>
+<label x="5.08" y="53.34" size="0.762" layer="95" rot="R180" xref="yes"/>
+</segment>
 </net>
 <net name="SDA" class="0">
@@
 <label x="99.06" y="78.74" size="1.778" layer="95" rot="R180" xref="yes"/>
 </segment>
+<segment>
+<wire x1="7.62" y1="55.88" x2="5.08" y2="55.88" width="0.1524" layer="91"/>
+<pinref part="U$1" gate="G$1" pin="6"/>
+<label x="5.08" y="55.88" size="0.762" layer="95" rot="R180" xref="yes"/>
+</segment>
 </net>
 <net name="HALL_A_R" class="0">
@@
 <label x="71.12" y="86.36" size="0.762" layer="95" rot="R180" xref="yes"/>
 </segment>
+<segment>
+<wire x1="7.62" y1="35.56" x2="5.08" y2="35.56" width="0.1524" layer="91"/>
+<pinref part="U$1" gate="G$1" pin="14"/>
+<label x="5.08" y="35.56" size="0.762" layer="95" rot="R180" xref="yes"/>
+</segment>
 </net>
 <net name="HALL_B_R" class="0">
@@
 <label x="71.12" y="83.82" size="0.762" layer="95" rot="R180" xref="yes"/>
 </segment>
+<segment>
+<wire x1="7.62" y1="33.02" x2="5.08" y2="33.02" width="0.1524" layer="91"/>
+<pinref part="U$1" gate="G$1" pin="15"/>
+<label x="5.08" y="33.02" size="0.762" layer="95" rot="R180" xref="yes"/>
+</segment>
 </net>
 <net name="HALL_A_L" class="0">
@@
 <label x="20.32" y="86.36" size="0.762" layer="95" rot="R180" xref="yes"/>
 </segment>
+<segment>
+<wire x1="7.62" y1="30.48" x2="5.08" y2="30.48" width="0.1524" layer="91"/>
+<pinref part="U$1" gate="G$1" pin="16"/>
+<label x="5.08" y="30.48" size="0.762" layer="95" rot="R180" xref="yes"/>
+</segment>
 </net>
 <net name="HALL_B_L" class="0">
@@
 <pinref part="P2" gate="G$1" pin="6"/>
 <label x="20.32" y="83.82" size="0.762" layer="95" rot="R180" xref="yes"/>
+</segment>
+<segment>
+<wire x1="7.62" y1="27.94" x2="5.08" y2="27.94" width="0.1524" layer="91"/>
+<pinref part="U$1" gate="G$1" pin="17"/>
+<label x="5.08" y="27.94" size="0.762" layer="95" rot="R180" xref="yes"/>
 </segment>
 </net>
@@
 </segment>
 </net>
+<net name="5.0V" class="0">
+<segment>
+<pinref part="X9" gate="-1" pin="S"/>
+<wire x1="256.54" y1="66.04" x2="254" y2="66.04" width="0.1524" layer="91"/>
+<wire x1="254" y1="66.04" x2="254" y2="78.74" width="0.1524" layer="91"/>
+<label x="254" y="78.74" size="1.778" layer="95" rot="R90" xref="yes"/>
+<pinref part="S2" gate="1" pin="P"/>
+<wire x1="254" y1="78.74" x2="269.24" y2="78.74" width="0.1524" layer="91"/>
+<wire x1="269.24" y1="78.74" x2="269.24" y2="76.2" width="0.1524" layer="91"/>
+</segment>
+</net>

Commit message: ボードのグランド以外を配置
Connections:
- removed net IO20: U$1.26
- removed net VCC: P1.3, P2.3, U$2.VCC, U$3.VCC, U$4.VIN
- new net IO12: U$1.16
- new net IO13: U$1.17
- net 3V3: now also P1.3, P2.3, U$2.VCC, U$3.VCC, X6-1.S
- net 3V3_EN: no longer X6-1.S
- net HALL_A_L: now also U$1.26; no longer U$1.16
- net HALL_B_L: now also U$1.27; no longer U$1.17
- net IO0: now also U$2.AIN2; no longer U$2.BIN1
- net IO1: now also U$2.BIN1; no longer U$2.AIN2
- net IO15: now also S1.P1
- net IO2: now also U$3.AIN2; no longer U$3.BIN1
- net IO21: no longer S1.P1, U$1.27
- net IO3: now also U$3.BIN1; no longer U$3.AIN2
- net MOTOR_A_L: now also U$2.AOUT2; no longer U$2.BOUT1
- net MOTOR_A_R: now also U$3.AOUT2; no longer U$3.BOUT1
- net MOTOR_B_L: now also U$2.BOUT1; no longer U$2.AOUT2
- net MOTOR_B_R: now also U$3.BOUT1; no longer U$3.AOUT2
- net VBUS: now also U$4.VIN

Commit message: 線を斜めに配置
Connections:
- net VBUS: no longer S2.S, TC4052DP.16, U$4.VIN, X5-1.S, X7-2.S
- net VSYS: now also S2.S, TC4052DP.16, U$4.VIN, X5-1.S, X7-2.S
Changed lines of the file:
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@@
 <label x="40.64" y="68.58" size="0.762" layer="95" xref="yes"/>
+</segment>
+</net>
+<net name="VSYS" class="2">
+<segment>
+<wire x1="40.64" y1="66.04" x2="38.1" y2="66.04" width="0.1524" layer="91"/>
+<pinref part="U$1" gate="G$1" pin="39"/>
+<label x="40.64" y="66.04" size="0.762" layer="95" xref="yes"/>
+</segment>
+<segment>
+<pinref part="U$4" gate="G$1" pin="VIN"/>
+<wire x1="78.74" y1="68.58" x2="71.12" y2="68.58" width="0.1524" layer="91"/>
+<wire x1="71.12" y1="68.58" x2="71.12" y2="71.12" width="0.1524" layer="91"/>
+<label x="71.12" y="71.12" size="1.778" layer="95" xref="yes"/>
 </segment>
 <segment>
@@
 <label x="274.32" y="86.36" size="1.778" layer="95" xref="yes"/>
 </segment>
-<segment>
-<pinref part="U$4" gate="G$1" pin="VIN"/>
-<wire x1="78.74" y1="68.58" x2="71.12" y2="68.58" width="0.1524" layer="91"/>
-<wire x1="71.12" y1="68.58" x2="71.12" y2="71.12" width="0.1524" layer="91"/>
-<label x="71.12" y="71.12" size="1.778" layer="95" xref="yes"/>
-</segment>
 </net>
-<net name="VSYS" class="2">
-<segment>
-<wire x1="40.64" y1="66.04" x2="38.1" y2="66.04" width="0.1524" layer="91"/>
-<pinref part="U$1" gate="G$1" pin="39"/>
-<label x="40.64" y="66.04" size="0.762" layer="95" xref="yes"/>
-</segment>
-</net>
