File: RoboKit/RoboKit.sch (EAGLE design)
At the start: 23 parts, among them CON1 XT30UPB-M, CON2 XT30UPB-M, P1 B6B-PH-K, P2 B6B-PH-K, U1 SSM6J808R, X1 JST-XH-06-PIN-LONG-PAD, X2 JST-XH-06-PIN-LONG-PAD

Commit message: :warning: Fix position of JLCPCB logo
Parts:
- removed C11, C2: 1uF, resistor:C-EUC0603
- removed C7: 0.1uF, SparkFun-Capacitors:4.7UF0603
- removed CON1, CON2: XT30UPB-M, XTn0 amass:XT30UPB-M
- removed R1, R4: 20k, SparkFun-Resistors:10KOHM-0603-1/10W-1%
- removed R5: 1k, Values of parts:POTTRS64W
- removed U$5: M51957, M51957B:M51957
- removed U$6: BSC093N04LSGATMA1, MOSFET_BSC093N04LSGATMA1:BSC093N04LSGATMA1
- removed U$7: FUSE, fuse:FUSE
- removed U$9: SW, akizuki sw:SW
- added C1: (no value), rcl:C-EU025-024X044
- added CONNECTOR1, CONNECTOR4, CONNECTOR5, CONNECTOR6: RESISTER, resistor:RESISTER
- added LED1, LED2: TLLY4400, led:TLLY4400
- added S2: (no value), switch-omron:40-XX
- added S3: (no value), switch-omron:10-XX
- added U$8: SW, akizuki sw:SW
- added X3, X4, X8: JST-XH-02-PIN-LONG-PAD, Rembrandt Electronics - JST XH Connectors v1-0:JST-XH-02-PIN-LONG-PAD
- added X5, X6: JST-XH-04-PIN-LONG-PAD, Rembrandt Electronics - JST XH Connectors v1-0:JST-XH-04-PIN-LONG-PAD
- added X7: JST-XH-10-PIN-LONG-PAD, Rembrandt Electronics - JST XH Connectors v1-0:JST-XH-10-PIN-LONG-PAD
- added X9: JST-XH-03-PIN-LONG-PAD, Rembrandt Electronics - JST XH Connectors v1-0:JST-XH-03-PIN-LONG-PAD
- R2: value 10k -> (none); device SparkFun-Resistors:1KOHM-0603-1/10W-1% -> rcl:R-US_R0603
- R3: value 2k -> (none); device SparkFun-Resistors:1KOHM-0603-1/10W-1% -> rcl:R-US_R0603
- U1: value SSM6J808R -> CD74HC4067SM96; device SSM6J808R:SSM6J808R -> CD74HC4067SM96:CD74HC4067SM96
- X1: value JST-XH-06-PIN-LONG-PAD -> JST-XH-03-PIN-LONG-PAD; device JST XH Connectors:JST-XH-06-PIN-LONG-PAD -> Rembrandt Electronics - JST XH Connectors v1-0:JST-XH-03-PIN-LONG-PAD
- X2: value JST-XH-06-PIN-LONG-PAD -> JST-XH-02-PIN-LONG-PAD; device JST XH Connectors:JST-XH-06-PIN-LONG-PAD -> Rembrandt Electronics - JST XH Connectors v1-0:JST-XH-02-PIN-LONG-PAD
Connections:
- net ADC1 renamed X-COM
- removed net +5V: X1-2.S, X2-2.S
- removed net ADC0: U$1.31
- removed net ADC2: U$1.34
- removed net GND_IN: C11.2, C2.2, C7.1, CON2.-, R2.1, R3.2, U$5.GND, U$6.S, U$9.1
- removed net IO10: U$1.14
- removed net IO11: U$1.15
- removed net IO21: U$1.27, U$1.29
- removed net IO4: U$1.6
- removed net IO5: U$1.7
- removed net LINE: X1-3.S, X2-3.S
- removed net MD_INA_L: U$2.AIN1, U$2.AIN2
- removed net MD_INA_R: U$3.AIN1, U$3.AIN2
- removed net MD_INB_L: U$2.BIN1, U$2.BIN2
- removed net MD_INB_R: U$3.BIN1, U$3.BIN2
- removed net MUX0: X1-4.S, X2-4.S
- removed net MUX1: X1-5.S, X2-5.S
- removed net MUX2: X1-6.S, X2-6.S
- removed net N$5: C11.1, U$5.C
- removed net N$6: C7.2, R2.2, U$5.OUT, U$6.GATE
- removed net N$7: R4.1, U$9.2, U1.G
- removed net VCC: P1.3, P2.3, U$2.VCC, U$3.VCC, U$4.VIN
- removed net VIN: CON2.+, R4.2, U1.D
- removed net V_HIGH: U$7.3, U$7.4, U1.S
- new net 0X: U1.I0, X7-1.S
- new net 0Y: U1.I4, X7-5.S
- new net 1X: U1.I1, X7-2.S
- new net 1Y: U1.I5, X7-6.S
- new net 2X: U1.I2, X7-3.S
- new net 2Y: U1.I6, X7-7.S
- new net 3X: U1.I3, X7-4.S
- new net 3Y: U1.I7, X7-8.S
- new net 5.0V: U$8.1, X9-1.S
- new net ANALOG: U$1.34, X1-3.S
- new net N$11: U1.I8
- new net N$12: U1.I9
- new net N$13: U1.I10
- new net N$14: U1.I11
- new net N$15: U1.I12
- new net N$16: U1.I13
- new net N$17: U1.I14
- new net N$18: U1.I15
- new net N$19: CONNECTOR4.2, U1.COMMON_I/O
- new net N$4: CONNECTOR6.2, U1.!E
- new net Y-COM: CONNECTOR4.1, CONNECTOR5.2, U$1.31
- net 3V3: now also CONNECTOR1.1, P1.3, P2.3, U$2.VCC, U$3.VCC, X6-1.S
- net GND: now also C1.2, CONNECTOR5.1, CONNECTOR6.1, LED1.C, LED2.C, S2.S1, S3.S1, U1.GND, X2-2.S, X5-4.S, X6-2.S, X7-10.S, X8-2.S, X9-2.S; no longer CON1.-, U$6.D, X2-1.S
- net HALL_A_L: now also U$1.14
- net HALL_A_R: now also U$1.27
- net HALL_B_L: now also U$1.15
- net HALL_B_R: now also U$1.29
- net IO0: now also U$2.AIN1, U$2.AIN2
- net IO1: now also U$2.BIN1, U$2.BIN2
- net IO13: now also R3.2
- net IO14: now also R2.2
- net IO15: now also S2.P1
- net IO16: now also U1.S0
- net IO17: now also U1.S1
- net IO18: now also U1.S2
- net IO19: now also U1.S3
- net IO2: now also U$3.AIN1, U$3.AIN2
- net IO20: now also X8-1.S
- net IO3: now also U$3.BIN1, U$3.BIN2
- net MOTOR_A_L: now also X3-1.S
- net MOTOR_A_R: now also X4-1.S
- net MOTOR_B_L: now also X3-2.S
- net MOTOR_B_R: now also X4-2.S
- net N$1: now also LED1.A, R2.1; no longer R5.OUT, U$5.IN
- net N$2: now also CONNECTOR1.2, S2.P; no longer R3.1, R5.VDD
- net N$3: now also LED2.A, R3.1; no longer R1.1, R5.VSS
- net RUN: now also S3.P1
- net SCL: now also U$1.7, X5-2.S, X6-4.S
- net SDA: now also U$1.6, X5-1.S, X6-3.S
- net VOUT: now also X2-1.S, X9-3.S; no longer C2.1, CON1.+, R1.2, U$5.V, U$7.1, U$7.2
- net VSYS: now also C1.1, U$4.VIN, U$8.2, U1.VCC, X1-2.S, X5-3.S, X7-9.S
Other:
- note removed: "M51957B"
- note removed: "delay"
- note removed: "mosfet"
- note removed: "スイッチ"
- moved on the sheet: X1-1, X1-2, X1-3, X2-1, X2-2
