File: RoboKit/RoboKit.brd (EAGLE design)
At the start: 134 x 82 mm, 32 parts, among them CON1 XT30UPB-M, CON2 XT30UPB-M, P1 B6B-PH-K, P2 B6B-PH-K, U1 SSM6J808R, X3 JST-XH-02-PIN-LONG-PAD, X4 JST-XH-02-PIN-LONG-PAD, X5 JST-XH-04-PIN-LONG-PAD, X6 JST-XH-04-PIN-LONG-PAD, X7 JST-XH-10-PIN-LONG-PAD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

Commit message: 5回目課題
Routing:
- net IO1: track 93.5 -> 73.6 mm
Changed lines of the file:
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@@
 <contactref element="U$2" pad="INB2"/>
 <contactref element="U$2" pad="INB1"/>
-<wire x1="51.435" y1="36.195" x2="50.165" y2="37.465" width="0.5" layer="1"/>
-<wire x1="50.165" y1="61.595" x2="50.165" y2="37.465" width="0.5" layer="1"/>
+<wire x1="51.435" y1="60.96" x2="50.8" y2="61.595" width="0.5" layer="1"/>
+<wire x1="50.165" y1="61.595" x2="50.8" y2="61.595" width="0.5" layer="1"/>
+<wire x1="51.435" y1="60.96" x2="51.435" y2="56.515" width="0.5" layer="1"/>
 <wire x1="51.435" y1="56.515" x2="50.165" y2="56.515" width="0.5" layer="1"/>
 <wire x1="69.315" y1="23.595" x2="74.9075" y2="23.595" width="0.5" layer="16"/>
-<wire x1="51.435" y1="56.515" x2="51.435" y2="36.195" width="0.5" layer="1"/>
-<wire x1="51.435" y1="36.195" x2="51.435" y2="28.8925" width="0.5" layer="1"/>
+<wire x1="51.435" y1="56.515" x2="51.435" y2="28.8925" width="0.5" layer="1"/>
 <wire x1="69.315" y1="23.595" x2="61.9125" y2="16.1925" width="0.5" layer="16"/>
 <via x="51.435" y="28.8925" extent="1-16" drill="0.35"/>
