File: RoboKit_2/RoboKit.brd (EAGLE design)
At the start: 134 x 82 mm, 28 parts, among them P1 B6B-PH-K, P2 B6B-PH-K, U1 CD74HC4067SM96, X1 JST-XH-03-PIN-LONG-PAD, X2 JST-XH-02-PIN-LONG-PAD, X3 JST-XH-02-PIN-LONG-PAD, X4 JST-XH-02-PIN-LONG-PAD, X5 JST-XH-04-PIN-LONG-PAD, X6 JST-XH-04-PIN-LONG-PAD, X7 JST-XH-10-PIN-LONG-PAD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

Commit message: とりあえず完成！
Parts:
- removed CONNECTOR2, CONNECTOR3: RESISTER, resistor:RESISTER_SOCKET
- added R2, R3: (no value), rcl:R0603
- moved X7 5.79 mm to (86.0, 14.6)
- moved LED2 4.85 mm to (12.1, 25.4), turned to 180 degrees
- moved LED1 4.26 mm to (12.1, 19.4), turned to 180 degrees
- moved X1 0.95 mm to (67.0, 8.89)
Connections:
- new net $10: C1.1, U1.24
- net 0X: now also X7.1; no longer X7.3
- net 0Y: now also X7.5; no longer X7.7
- net 1X: now also X7.2; no longer X7.4
- net 1Y: now also X7.6; no longer X7.8
- net 2X: now also X7.3; no longer X7.5
- net 2Y: now also X7.7; no longer X7.9
- net 3X: now also X7.4; no longer X7.6
- net 3Y: now also X7.8; no longer X7.10
- net GND: now also X7.10; no longer X7.1
- net HALL_A_L: now also U$1.14; no longer U$1.27
- net HALL_A_R: now also U$1.27; no longer U$1.14
- net HALL_B_L: now also U$1.15; no longer U$1.29
- net HALL_B_R: now also U$1.29; no longer U$1.15
- net IO13: now also R3.2; no longer CONNECTOR3.2
- net IO14: now also R2.2; no longer CONNECTOR2.2
- net IO20: now also X8.1
- net IO7: no longer X8.1
- net N$1: now also R2.1; no longer CONNECTOR2.1
- net N$3: now also R3.1; no longer CONNECTOR3.1
- net VSYS: now also X7.9; no longer C1.1, U1.24, X7.2
Routing:
- net GND: track 17.8 -> 506.0 mm, vias 0 -> 6
- net VOUT: track 2.22 -> 220.1 mm, vias 0 -> 4
- net VSYS: track 0.00 -> 204.5 mm
- net SDA: track 0.00 -> 176.6 mm, vias 0 -> 2
- net SCL: track 0.00 -> 164.3 mm, vias 0 -> 2
- net 3V3: track 32.1 -> 133.3 mm
- net IO3: track 14.4 -> 89.1 mm, vias 0 -> 1
- net RUN: track 0.00 -> 71.9 mm, vias 0 -> 3
- net ANALOG: track 0.00 -> 68.5 mm, vias 0 -> 1
- net IO2: track 23.1 -> 91.5 mm, vias 1 -> 2
- net MOTOR_B_L: track 0.00 -> 49.9 mm
- net MOTOR_A_L: track 0.00 -> 44.5 mm
- net Y-COM: track 0.00 -> 42.3 mm
- net HALL_B_L: track 0.00 -> 41.3 mm
- net HALL_A_L: track 0.00 -> 40.4 mm
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- added copper zone on layer 1, net 3V3
- added copper zone on layer 1, net 5.0V
- added copper zone on layer 1, net VOUT
- added copper zone on layer 16, net VSYS
Other:
- outline, holes or cut-outs redrawn

Commit message: かんせい
Parts:
- moved R2 34.6 mm to (19.7, 19.4)
- moved R3 34.6 mm to (19.7, 22.9)
Routing:
- net IO14: track 25.1 -> 40.2 mm
- net IO13: track 30.4 -> 40.8 mm
- net N$1: track 0.00 -> 5.50 mm
- net N$3: track 4.39 -> 6.77 mm
Changed lines of the file:
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@@
 <attribute name="VALUE" x="85.217" y="28.1305" size="1.27" layer="27" ratio="10"/>
 </element>
-<element name="R3" library="rcl" package="R0603" value="" x="1.5875" y="-6.6675" smashed="yes">
-<attribute name="NAME" x="0.9525" y="-6.0325" size="1.27" layer="25"/>
-<attribute name="VALUE" x="0.9525" y="-8.5725" size="1.27" layer="27"/>
+<element name="R3" library="rcl" package="R0603" value="" x="19.685" y="22.86" smashed="yes">
+<attribute name="NAME" x="19.05" y="23.495" size="1.27" layer="25"/>
+<attribute name="VALUE" x="19.05" y="20.955" size="1.27" layer="27"/>
 </element>
-<element name="R2" library="rcl" package="R0603" value="" x="1.5875" y="-10.16" smashed="yes">
-<attribute name="NAME" x="0.9525" y="-9.525" size="1.27" layer="25"/>
-<attribute name="VALUE" x="0.9525" y="-12.065" size="1.27" layer="27"/>
+<element name="R2" library="rcl" package="R0603" value="" x="19.685" y="19.3675" smashed="yes">
+<attribute name="NAME" x="19.05" y="20.0025" size="1.27" layer="25"/>
+<attribute name="VALUE" x="19.05" y="17.4625" size="1.27" layer="27"/>
 </element>
 </elements>
@@
 <wire x1="81.28" y1="69.85" x2="80.9625" y2="69.5325" width="0.5" layer="1"/>
 <wire x1="80.9625" y1="69.5325" x2="80.9625" y2="59.055" width="0.5" layer="1"/>
-<wire x1="88.5825" y1="49.8475" x2="89.535" y2="50.8" width="0.5" layer="1"/>
+<wire x1="88.265" y1="49.53" x2="89.535" y2="50.8" width="0.5" layer="1"/>
 <wire x1="80.9625" y1="59.055" x2="79.375" y2="57.4675" width="0.5" layer="1"/>
-<wire x1="79.375" y1="50.4825" x2="80.01" y2="49.8475" width="0.5" layer="1"/>
+<wire x1="79.375" y1="50.4825" x2="80.3275" y2="49.53" width="0.5" layer="1"/>
 <wire x1="79.375" y1="57.4675" x2="79.375" y2="50.4825" width="0.5" layer="1"/>
-<wire x1="80.01" y1="49.8475" x2="88.5825" y2="49.8475" width="0.5" layer="1"/>
+<wire x1="80.3275" y1="49.53" x2="88.265" y2="49.53" width="0.5" layer="1"/>
 </signal>
 <signal name="GND">
@@
 <wire x1="90.4875" y1="41.275" x2="91.495" y2="40.2675" width="1" layer="1"/>
 <wire x1="91.495" y1="34.6075" x2="91.495" y2="38.4175" width="1" layer="16"/>
-<wire x1="10.795" y1="19.3675" x2="10.795" y2="25.4" width="1" layer="1"/>
-<wire x1="10.795" y1="19.3675" x2="10.795" y2="16.8275" width="1" layer="1"/>
-<wire x1="10.795" y1="16.8275" x2="23.1775" y2="16.8275" width="1" layer="1"/>
-<wire x1="23.1775" y1="16.8275" x2="23.1775" y2="26.035" width="1" layer="1"/>
+<wire x1="10.795" y1="19.3675" x2="10.795" y2="25.4" width="1" layer="16"/>
+<wire x1="10.795" y1="19.3675" x2="10.795" y2="16.8275" width="1" layer="16"/>
+<wire x1="10.795" y1="16.8275" x2="23.1775" y2="16.8275" width="1" layer="16"/>
+<wire x1="23.1775" y1="16.8275" x2="23.1775" y2="26.035" width="1" layer="16"/>
 <wire x1="23.1775" y1="26.035" x2="23.1775" y2="31.75" width="1" layer="1"/>
 <wire x1="25.7175" y1="34.29" x2="48.26" y2="34.29" width="1" layer="1"/>
@@
 <wire x1="59.3725" y1="16.51" x2="58.7375" y2="15.875" width="1" layer="16"/>
 <wire x1="58.7375" y1="15.875" x2="56.8325" y2="15.875" width="1" layer="16"/>
-<wire x1="56.8325" y1="15.875" x2="56.515" y2="15.875" width="1" layer="16"/>
 <via x="56.8325" y="15.875" extent="1-16" drill="0.8"/>
 <via x="58.7375" y="15.875" extent="1-16" drill="0.8"/>
@@
 <signal name="IO14">
 <contactref element="U$1" pad="19"/>
-<wire x1="33.69" y1="23.395" x2="58.76" y2="23.395" width="0.5" layer="1"/>
+<wire x1="33.69" y1="23.395" x2="33.9725" y2="23.395" width="0.5" layer="1"/>
 <contactref element="R2" pad="2"/>
-<wire x1="2.4375" y1="-10.16" x2="33.69" y2="23.395" width="0" layer="19" extent="1-1"/>
+<wire x1="25.404375" y1="23.395" x2="33.69" y2="23.395" width="0.5" layer="1"/>
+<wire x1="33.9725" y1="23.395" x2="58.76" y2="23.395" width="0.5" layer="1"/>
+<wire x1="20.535" y1="19.3675" x2="22.38375" y2="19.3675" width="0.5" layer="1"/>
+<wire x1="22.38375" y1="19.3675" x2="25.404375" y2="23.395" width="0.5" layer="1"/>
 </signal>
 <signal name="IO15">
@@
 <vertex x="85.09" y="70.8025"/>
 </polygon>
+<polygon width="0.5" layer="1">
+<vertex x="32.0675" y="50.4825"/>
+<vertex x="42.8625" y="50.4825"/>
+<vertex x="44.1325" y="51.435"/>
+<vertex x="44.1325" y="53.0225"/>
+<vertex x="42.8625" y="53.975"/>
+<vertex x="38.1" y="53.975"/>
+<vertex x="36.195" y="56.515"/>
+<vertex x="34.29" y="56.515"/>
+<vertex x="33.655" y="57.15"/>
+<vertex x="33.655" y="69.5325"/>
+<vertex x="32.7025" y="70.485"/>
+<vertex x="30.48" y="68.58"/>
+<vertex x="30.48" y="50.4825"/>
+</polygon>
 </signal>
 <signal name="ANALOG">
@@
 <wire x1="42.545" y1="69.215" x2="42.545" y2="73.66" width="1.8" layer="16"/>
 <via x="32.385" y="73.66" extent="1-16" drill="0.8"/>
-<wire x1="42.8625" y1="73.66" x2="42.545" y2="73.66" width="1.8" layer="16"/>
 <wire x1="42.545" y1="73.66" x2="32.385" y2="73.66" width="1.8" layer="16"/>
-<wire x1="42.545" y1="73.66" x2="44.1325" y2="73.66" width="1.8" layer="1"/>
-<wire x1="44.1325" y1="73.66" x2="50.8" y2="80.3275" width="1.8" layer="1"/>
+<wire x1="50.8" y1="80.3275" x2="44.1325" y2="73.66" width="1.8" layer="1"/>
 <wire x1="82.2325" y1="80.3275" x2="50.8" y2="80.3275" width="1.8" layer="1"/>
 <wire x1="84.455" y1="78.74" x2="82.8675" y2="80.3275" width="1.8" layer="16"/>
@@
 </polygon>
 <via x="84.455" y="77.1525" extent="1-16" drill="1"/>
+<wire x1="44.1325" y1="73.66" x2="42.545" y2="73.66" width="1.8" layer="1"/>
 </signal>
 <signal name="2X">
@@
 <contactref element="U$1" pad="17"/>
 <wire x1="58.76" y1="28.475" x2="58.6375" y2="28.475" width="0.5" layer="1"/>
-<wire x1="54.9275" y1="24.765" x2="33.02" y2="24.765" width="0.5" layer="1"/>
-<wire x1="33.02" y1="24.765" x2="30.7975" y2="22.5425" width="0.5" layer="1"/>
 <wire x1="58.6375" y1="28.475" x2="54.9275" y2="24.765" width="0.5" layer="1"/>
 <contactref element="R3" pad="2"/>
-<wire x1="2.4375" y1="-6.6675" x2="30.7975" y2="22.5425" width="0" layer="19" extent="1-1"/>
+<wire x1="54.9275" y1="24.765" x2="24.4475" y2="24.765" width="0.5" layer="1"/>
+<wire x1="24.4475" y1="24.765" x2="23.1775" y2="22.86" width="0.5" layer="1"/>
+<wire x1="23.1775" y1="22.86" x2="20.535" y2="22.86" width="0.5" layer="1"/>
 </signal>
 <signal name="IO12">
@@
 <contactref element="LED1" pad="A"/>
 <contactref element="R2" pad="1"/>
-<wire x1="0.7375" y1="-10.16" x2="13.335" y2="19.3675" width="0" layer="19" extent="1-1"/>
+<wire x1="13.335" y1="19.3675" x2="18.835" y2="19.3675" width="0.5" layer="1"/>
 </signal>
 <signal name="N$3">
 <contactref element="LED2" pad="A"/>
-<wire x1="17.725" y1="25.4" x2="13.335" y2="25.4" width="0.5" layer="1"/>
 <contactref element="R3" pad="1"/>
-<wire x1="0.7375" y1="-6.6675" x2="13.335" y2="25.4" width="0" layer="19" extent="1-1"/>
+<wire x1="18.835" y1="22.86" x2="15.24" y2="22.86" width="0.5" layer="1"/>
+<wire x1="15.24" y1="22.86" x2="13.335" y2="25.4" width="0.5" layer="1"/>
 </signal>
 <signal name="N$4">
