File: RoboKit_2/RoboKit.sch (EAGLE design)
At the start: 28 parts, among them P1 B6B-PH-K, P2 B6B-PH-K, U1 CD74HC4067SM96, X1 JST-XH-03-PIN-LONG-PAD, X2 JST-XH-02-PIN-LONG-PAD, X3 JST-XH-02-PIN-LONG-PAD, X4 JST-XH-02-PIN-LONG-PAD, X5 JST-XH-04-PIN-LONG-PAD, X6 JST-XH-04-PIN-LONG-PAD, X7 JST-XH-10-PIN-LONG-PAD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

Commit message: とりあえず完成！
Parts:
- removed CONNECTOR2, CONNECTOR3: RESISTER, resistor:RESISTER
- added R2, R3: (no value), rcl:R-US_R0603
Connections:
- new net $10: C1.1, U1.VCC
- net 0X: now also X7-1.S; no longer X7-3.S
- net 0Y: now also X7-5.S; no longer X7-7.S
- net 1X: now also X7-2.S; no longer X7-4.S
- net 1Y: now also X7-6.S; no longer X7-8.S
- net 2X: now also X7-3.S; no longer X7-5.S
- net 2Y: now also X7-7.S; no longer X7-9.S
- net 3X: now also X7-4.S; no longer X7-6.S
- net 3Y: now also X7-8.S; no longer X7-10.S
- net GND: now also X7-10.S; no longer X7-1.S
- net HALL_A_L: now also U$1.14; no longer U$1.27
- net HALL_A_R: now also U$1.27; no longer U$1.14
- net HALL_B_L: now also U$1.15; no longer U$1.29
- net HALL_B_R: now also U$1.29; no longer U$1.15
- net IO13: now also R3.2; no longer CONNECTOR3.2
- net IO14: now also R2.2; no longer CONNECTOR2.2
- net IO20: now also X8-1.S
- net IO7: no longer X8-1.S
- net N$1: now also R2.1; no longer CONNECTOR2.1
- net N$3: now also R3.1; no longer CONNECTOR3.1
- net VSYS: now also X7-9.S; no longer C1.1, U1.VCC, X7-2.S

Commit message: マルチプレクサの電源回り付近を修正
Connections:
- removed net $10: C1.1, U1.VCC
- net VSYS: now also C1.1, U1.VCC
Changed lines of the file:
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@@
 <label x="190.5" y="109.22" size="1.778" layer="95" rot="R180" xref="yes"/>
+</segment>
+<segment>
+<pinref part="U1" gate="G$1" pin="VCC"/>
+<wire x1="279.4" y1="198.12" x2="281.94" y2="198.12" width="0.1524" layer="91"/>
+<label x="281.94" y="198.12" size="1.778" layer="95" xref="yes"/>
+<pinref part="C1" gate="G$1" pin="1"/>
 </segment>
 </net>
@@
 </segment>
 </net>
-<net name="$10" class="2">
-<segment>
-<pinref part="U1" gate="G$1" pin="VCC"/>
-<wire x1="279.4" y1="198.12" x2="281.94" y2="198.12" width="0.1524" layer="91"/>
-<label x="281.94" y="198.12" size="1.778" layer="95" xref="yes"/>
-<pinref part="C1" gate="G$1" pin="1"/>
-</segment>
-</net>

Commit message: XH10ピンが刺さらない不具合を修正し、アナログ出力の印刷が逆になっていたのを修正し、ver2.0のシルクを追加
Connections:
- removed net ADC2: U$1.34
- new net ADC_VREF: U$1.35
- net ANALOG: now also U$1.34, X1-3.S; no longer U$1.35, X1-1.S
- net GND: now also X1-1.S; no longer X1-3.S
Changed lines of the file:
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@@
-</segment>
-<segment>
-<pinref part="X1" gate="-3" pin="S"/>
-<wire x1="71.12" y1="38.1" x2="68.58" y2="38.1" width="0.1524" layer="91"/>
-<label x="68.58" y="38.1" size="1.778" layer="95" rot="R180" xref="yes"/>
 </segment>
 <segment>
@@
 <wire x1="193.04" y1="106.68" x2="190.5" y2="106.68" width="0.1524" layer="91"/>
 <label x="190.5" y="106.68" size="1.778" layer="95" rot="R180" xref="yes"/>
+</segment>
+<segment>
+<pinref part="X1" gate="-1" pin="S"/>
+<wire x1="71.12" y1="43.18" x2="68.58" y2="43.18" width="0.1524" layer="91"/>
+<label x="68.58" y="43.18" size="1.778" layer="95" rot="R180" xref="yes"/>
 </segment>
 </net>
@@
 <net name="ANALOG" class="0">
 <segment>
-<wire x1="40.64" y1="55.88" x2="38.1" y2="55.88" width="0.1524" layer="91"/>
-<pinref part="U$1" gate="G$1" pin="35"/>
-<label x="40.64" y="55.88" size="0.762" layer="95" xref="yes"/>
-</segment>
-<segment>
-<pinref part="X1" gate="-1" pin="S"/>
-<wire x1="71.12" y1="43.18" x2="68.58" y2="43.18" width="0.1524" layer="91"/>
-<label x="68.58" y="43.18" size="1.778" layer="95" rot="R180" xref="yes"/>
-</segment>
-</net>
-<net name="ADC2" class="0">
-<segment>
 <wire x1="40.64" y1="53.34" x2="38.1" y2="53.34" width="0.1524" layer="91"/>
 <pinref part="U$1" gate="G$1" pin="34"/>
 <label x="40.64" y="53.34" size="0.762" layer="95" xref="yes"/>
+</segment>
+<segment>
+<pinref part="X1" gate="-3" pin="S"/>
+<wire x1="71.12" y1="38.1" x2="68.58" y2="38.1" width="0.1524" layer="91"/>
+<label x="68.58" y="38.1" size="1.778" layer="95" rot="R180" xref="yes"/>
 </segment>
 </net>
@@
 </segment>
 </net>
+<net name="ADC_VREF" class="0">
+<segment>
+<wire x1="40.64" y1="55.88" x2="38.1" y2="55.88" width="0.1524" layer="91"/>
+<pinref part="U$1" gate="G$1" pin="35"/>
+<label x="40.64" y="55.88" size="0.762" layer="95" xref="yes"/>
+</segment>
+</net>
